File: pcbs/left/left.kicad_pcb (KiCad board)
At the start: 2 copper layers, 90 x 73 mm, 28 parts, among them J1 Conn_01x10_Socket

Commit message: plate and pcb finished
Connections:
- J1 pad 10: C5 -> C6
- J1 pad 5: C0 -> C1
- J1 pad 6: C1 -> C2
- J1 pad 7: C2 -> C3
- J1 pad 8: C3 -> C4
- J1 pad 9: C4 -> C5
Routing:
- net C5: track 0.00 -> 149.4 mm
- net R1: track 0.00 -> 139.0 mm
- net C4: track 0.00 -> 106.7 mm
- net R2: track 0.00 -> 104.4 mm
- net R3: track 0.00 -> 81.3 mm
- net C3: track 0.00 -> 56.3 mm
- net C2: track 0.00 -> 38.8 mm
- net C1: track 0.00 -> 35.0 mm
- net middle_top: track 0.00 -> 12.9 mm
- net middle_bottom: track 0.00 -> 12.6 mm
- net ring_bottom: track 0.00 -> 12.5 mm
- net inner_thumb: track 0.00 -> 12.5 mm
- net inner_bottom: track 0.00 -> 12.5 mm
- net index_top: track 0.00 -> 12.5 mm
- net pinky_top: track 0.00 -> 12.5 mm
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- added copper zone on B.Cu, net GND
- added copper zone on F.Cu, net GND
Other:
- net class Default removed
