File: pcbs/right/right.kicad_pcb (KiCad board)
At the start: 2 copper layers, 108 x 73 mm, 32 parts, among them J1 Conn_01x10_Socket

Commit message: plate and pcb finished
Connections:
- J1 pad 10: C5 -> C6
- J1 pad 5: C0 -> C1
- J1 pad 6: C1 -> C2
- J1 pad 7: C2 -> C3
- J1 pad 8: C3 -> C4
- J1 pad 9: C4 -> C5
- S1 pad 1: C0 -> C6
- S10 pad 1: C4 -> C2
- S11 pad 1: C5 -> C1
- S12 pad 1: C5 -> C1
- S13 pad 1: C4 -> C2
- S14 pad 1: C5 -> C1
- S2 pad 1: C0 -> C6
- S3 pad 1: C1 -> C5
- S4 pad 1: C1 -> C5
- S5 pad 1: C2 -> C4
- S6 pad 1: C2 -> C4
- S9 pad 1: C4 -> C2
- _1 pad 1: R1 -> R3
- _3 pad 1: R3 -> R1
Routing:
- net R1: track 0.00 -> 179.6 mm
- net C1: track 0.00 -> 160.1 mm
- net R2: track 0.00 -> 124.8 mm
- net C2: track 0.00 -> 90.1 mm
- net R3: track 0.00 -> 89.9 mm
- net C6: track 0.00 -> 62.3 mm
- net C5: track 0.00 -> 44.5 mm
- net C3: track 0.00 -> 43.0 mm
- net C4: track 0.00 -> 40.8 mm
- net mirror_ext_top: track 0.00 -> 13.5 mm
- net mirror_ext_bottom: track 0.00 -> 12.8 mm
- net mirror_outer_thumb: track 0.00 -> 12.8 mm
- net mirror_middle_top: track 0.00 -> 12.7 mm
- net mirror_middle_bottom: track 0.00 -> 12.7 mm
- net mirror_inner_thumb: track 0.00 -> 12.7 mm
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- added copper zone on B.Cu, net GND
- added copper zone on F.Cu, net GND
Other:
- net class Default removed
